File: A65_Assemble/A65.kicad_pcb (KiCad board)
At the start: 2 copper layers, 304.4 x 98.8 mm, 137 parts, among them J1 Conn_01x02, SW1 SW_PUSH, SW10 SW_PUSH, SW11 SW_PUSH, SW12 SW_PUSH, SW13 SW_PUSH, SW14 SW_PUSH, SW15 SW_PUSH, SW16 SW_PUSH, SW17 SW_PUSH, SW18 SW_PUSH, SW19 SW_PUSH, SW2 SW_PUSH, SW20 SW_PUSH, SW21 SW_PUSH, SW22 SW_PUSH, SW23 SW_PUSH, SW24 SW_PUSH, SW25 SW_PUSH, SW26 SW_PUSH, SW27 SW_PUSH, SW28 SW_PUSH, SW29 SW_PUSH, SW3 SW_PUSH, SW30 SW_PUSH, SW31 SW_PUSH, SW32 SW_PUSH, SW33 SW_PUSH, SW34 SW_PUSH, SW35 SW_PUSH, SW36 SW_PUSH, SW37 SW_PUSH, SW38 SW_PUSH, SW39 SW_PUSH, SW4 SW_PUSH, SW40 SW_PUSH, SW41 SW_PUSH, SW42 SW_PUSH, SW43 SW_PUSH, SW44 SW_PUSH, SW45 SW_PUSH, SW46 SW_PUSH, SW47 SW_PUSH, SW48 SW_PUSH, SW49 SW_PUSH, SW5 SW_PUSH, SW50 SW_PUSH, SW51 SW_PUSH, SW52 SW_PUSH, SW53 SW_PUSH, SW54 SW_PUSH, SW55 SW_PUSH, SW56 SW_PUSH, SW57 SW_PUSH, SW58 SW_PUSH, SW59 SW_PUSH, SW6 SW_PUSH, SW60 SW_PUSH, SW61 SW_PUSH, SW62 SW_PUSH, SW63 SW_PUSH, SW64 SW_PUSH, SW65 SW_PUSH, SW66 SW_PUSH, SW67 SW_PUSH, SW68 SW_PUSH, SW7 SW_PUSH, SW8 SW_PUSH, SW9 SW_PUSH, U1 BLEMicroPro

Commit message: Fixed reset switch position.
Parts:
- moved SW68 14.7 mm to (280.5, 42.6), turned to 0 degrees
- moved D64 4.76 mm to (313.1, 31.5)
- moved D62 4.65 mm to (279.0, 37.2), turned to 180 degrees
Routing:
- net Col1: track 467.9 -> 449.8 mm, vias 2 -> 0
- net Row0: track 361.3 -> 343.2 mm, vias 3 -> 2
- net Col3: track 493.4 -> 477.8 mm, vias 2 -> 1
- net Col2: track 452.6 -> 438.2 mm, vias 2 -> 0
- net Col0: track 518.3 -> 505.6 mm
- net Reset: track 22.2 -> 34.6 mm
- net GND: track 170.1 -> 181.7 mm
- net Col5: track 332.0 -> 340.2 mm, vias 2 -> 3
- net Col4: track 421.5 -> 414.4 mm, vias 1 -> 3
- net Col6: track 336.8 -> 335.7 mm
- net Col7: track 307.4 -> 308.4 mm
- net Row1: vias 1 -> 0
Other:
- board text added: "MALIC ACID A65 rev1.0 Designed by NINETH SKY Studio"
- board text removed: "MALIC ACID A65 rev0.1 Designed by NINETH SKY Studio"
